Commit message: Some minor modifications for the Mercury test environment

File: urdf/sample.urdf (robot description, URDF)
Before this commit: robot dummy_robot, 4 links, 3 joints
Links:
- removed link end_link
- removed link second_middle_link
Joints:
- removed joint arm_joint_2
- removed joint arm_joint_3
